File: 8bit_CPU-V0_1/ADD_register.kicad_sch (KiCad schematic)
At the start: 17 parts, among them U22 74LS04, U24 74LS08, U30 74LS32, U33 74LS04, U35 74LS574, U36 74LS08, U37 74LS08, U44 74LS04, U6 74LS245

Commit message: Refining schematics
Parts:
- added D1, D2, D3, D4, D5, D6, D7, D8: LED, symbol Device:LED
- added RN1: 330, Resistor_THT:R_Array_SIP11, symbol Device:R_Network10_US
- renumbered U35 to U41
Connections:
- net GND: now also RN1.1 (common)
- net at U36.12, U41.12 (Q7), U6.9 (A7): now also D8.2 (A)
- net at U36.9, U41.13 (Q6), U6.8 (A6): now also D7.2 (A)
- net at U37.4, U41.14 (Q5), U6.7 (A5): now also D6.2 (A)
- net at U37.1, U41.15 (Q4), U6.6 (A4): now also D5.2 (A)
- net at U24.12, U41.16 (Q3), U6.5 (A3): now also D4.2 (A)
- net at U24.9, U41.17 (Q2), U6.4 (A2): now also D3.2 (A)
- net at U36.4, U41.18 (Q1), U6.3 (A1): now also D2.2 (A)
- net at U36.1, U41.19 (Q0), U6.2 (A0): now also D1.2 (A)
- new net: D1.1 (K), RN1.11 (R10)
- new net: D8.1 (K), RN1.2 (R1)
- new net: D2.1 (K), RN1.10 (R9)
- new net: D7.1 (K), RN1.3 (R2)
- new net: D6.1 (K), RN1.4 (R3)
- new net: D5.1 (K), RN1.5 (R4)
- new net: D4.1 (K), RN1.8 (R7)
- new net: D3.1 (K), RN1.9 (R8)
Other:
- moved on the sheet: C1, C6, U22B, U24C, U24D, U30A, U33G, U35E, U36A, U36B, U36C, U36D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

Commit message: update.
Parts:
- removed C1: 0.1uF, symbol Device:C
- removed U35: 74LS32, symbol 74xx:74LS32
- added unit 5 of U41
- renumbered U41 to U33, U22 to U38, U44 to U38, U33 to U38, U37 to U39, U36 to U39, U36 to U40, U24 to U40, U37 to U40, U30 to U41
Connections:
- net ADD/ADL: now also U38.11; no longer U38.1
- net ADD/SB(0-6): now also U39.10, U39.13, U39.5, U40.10, U40.13, U40.2, U40.5, U41.9; no longer U39.10, U39.2, U39.5, U40.10, U40.13, U40.2, U40.5, U41.1
- net ADD/SB(7): now also U39.2, U41.10; no longer U39.13, U41.2
- net at D8.2 (A), U33.12 (Q7), U6.9 (A7): now also U39.1; no longer U39.12
- net at D7.2 (A), U33.13 (Q6), U6.8 (A6): now also U39.4; no longer U39.9
- net at D6.2 (A), U33.14 (Q5), U6.7 (A5): now also U39.12; no longer U39.4
- net at D5.2 (A), U33.15 (Q4), U6.6 (A4): now also U39.9; no longer U39.1
- net at D4.2 (A), U33.16 (Q3), U6.5 (A3): now also U40.1; no longer U40.12
- net at D3.2 (A), U33.17 (Q2), U6.4 (A2): now also U40.4; no longer U40.9
- net at D2.2 (A), U33.18 (Q1), U6.3 (A1): now also U40.12; no longer U40.4
- net at D1.2 (A), U33.19 (Q0), U6.2 (A0): now also U40.9; no longer U40.1
- net at U6.19 (CE): now also U38.8; no longer U38.4
- net at U6.2 (A0): now also U40.8; no longer U40.3
- net at U6.3 (A1): now also U40.11; no longer U40.6
- net at U6.4 (A2): now also U40.6; no longer U40.8
- net at U6.5 (A3): now also U40.3; no longer U40.11
- net at U6.6 (A4): now also U39.8; no longer U39.3
- net at U6.7 (A5): now also U39.11; no longer U39.6
- net at U6.8 (A6): now also U39.6; no longer U39.8
- net at U6.9 (A7): now also U39.3; no longer U39.11
- net at U6.19 (CE): now also U38.10; no longer U38.2
- new net: U38.9, U41.8
