File: 8bit_CPU-V0_1/AInput_reg.kicad_sch (KiCad schematic)
At the start: 19 parts, among them U13 74LS04, U3 74LS173, U4 74LS173, U6 74LS245, U9 74LS32

Commit message: Modifications
-Nammed sub parts of circuits
-Created new prepared sheets for ALU ANDS and EORS
Parts:
- removed C1: 0.1uF, symbol Device:C
- removed unit 7 of U13
- renumbered U13 to U5
Connections:
- net SB/ADD: now also U5.13; no longer U5.5
- net ~{Ain_RST}: now also U5.9; no longer U5.1
- net at U3.15 (Mr), U4.15 (Mr): now also U5.8; no longer U5.2
- net at U6.19 (CE): now also U5.12; no longer U5.6
- net at U3.10 (E2), U3.9 (E1), U4.10 (E2)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: now also U5.10; no longer U5.4
- net at U9.3: now also U5.11; no longer U5.3

Commit message: ALU finished
Parts:
- added C7: 0.1uF, symbol Device:C
- added U7: 74HCT04, symbol 74xx:74HCT04
- renumbered U5 to U13
Connections:
- net GND: now also C7.2, U7.7 (GND)
- net SB/ADD: now also U13.1; no longer U13.13
- net VCC: now also C7.1, U7.14 (VCC)
- net ~{Ain_RST}: now also U13.5; no longer U13.9
- net at U3.15 (Mr), U4.15 (Mr): now also U13.6; no longer U13.8
- net at U6.19 (CE): now also U13.2; no longer U13.12
- net at U3.10 (E2), U3.9 (E1), U4.10 (E2)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: now also U13.4; no longer U13.10
- net at U9.3: now also U13.3; no longer U13.11
Other:
- note added: "24 AWG"
- note added: "Test Switch #1"
- note added: "Test Switch #2"
- company: (none) -> PRP-DIY
- title: (none) -> PRP-6502 -- ALU : B Input Register
- moved on the sheet: U13C

Commit message: Refining schematics
Other:
- title: PRP-6502 -- ALU : B Input Register -> PRP-6502 -- ALU : A Input Register
Changed lines of the file:
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@@
   (paper "A4")
   (title_block
-    (title "PRP-6502 -- ALU : B Input Register")
+    (title "PRP-6502 -- ALU : A Input Register")
     (date "2023-07-02")
     (company "PRP-DIY")

Commit message: update.
Parts:
- renumbered U13 to U9
Changed lines of the file:
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@@
   (title_block
     (title "PRP-6502 -- ALU : A Input Register")
-    (date "2023-07-02")
+    (date "2023-07-06")
+    (rev "1")
     (company "PRP-DIY")
   )
@@
   )
   (wire (pts (xy 160.02 125.73) (xy 160.02 153.67))
-    (stroke (width 0) (type default))
-  )
-  (wire (pts (xy 67.31 85.09) (xy 71.12 85.09))
     (stroke (width 0) (type default))
   )
@@
         )
         (path "/81b49a11-4d6c-4532-89fe-728a8cf00278/25bbece4-880f-4fa1-94ee-76ee775f4584"
-          (reference "U13") (unit 7)
+          (reference "U9") (unit 7)
         )
       )
@@
   (symbol (lib_id "74xx:74LS04") (at 55.88 153.67 0) (unit 3)
     (in_bom yes) (on_board yes) (dnp no)
-    (property "Reference" "U13" (at 54.61 153.67 0)
+    (property "Reference" "U9" (at 54.61 153.67 0)
       (effects (font (size 1.27 1.27)))
     )
@@
       (project "8bit_CPU-V0_1"
         (path "/81b49a11-4d6c-4532-89fe-728a8cf00278/25bbece4-880f-4fa1-94ee-76ee775f4584"
-          (reference "U13") (unit 3)
+          (reference "U9") (unit 3)
         )
       )
@@
     )
   )
-  (symbol (lib_id "power:GND") (at 67.31 85.09 0) (unit 1)
-    (in_bom yes) (on_board yes) (dnp no)
-    (property "Reference" "#PWR021" (at 67.31 91.44 0)
-      (effects (font (size 1.27 1.27)) hide)
-    )
-    (property "Value" "GND" (at 67.31 88.9 0)
-      (effects (font (size 1.27 1.27)))
-    )
-    (property "Footprint" "" (at 67.31 85.09 0)
-      (effects (font (size 1.27 1.27)) hide)
-    )
-    (property "Datasheet" "" (at 67.31 85.09 0)
+  (symbol (lib_id "power:GND") (at 71.12 85.09 0) (unit 1)
+    (in_bom yes) (on_board yes) (dnp no)
+    (property "Reference" "#PWR021" (at 71.12 91.44 0)
+      (effects (font (size 1.27 1.27)) hide)
+    )
+    (property "Value" "GND" (at 71.12 88.9 0)
+      (effects (font (size 1.27 1.27)))
+    )
+    (property "Footprint" "" (at 71.12 85.09 0)
+      (effects (font (size 1.27 1.27)) hide)
+    )
+    (property "Datasheet" "" (at 71.12 85.09 0)
       (effects (font (size 1.27 1.27)) hide)
     )
@@
   (symbol (lib_id "74xx:74LS04") (at 54.61 106.68 90) (unit 1)
     (in_bom yes) (on_board yes) (dnp no)
-    (property "Reference" "U13" (at 54.61 107.95 0)
+    (property "Reference" "U9" (at 54.61 107.95 0)
       (effects (font (size 1.27 1.27)))
     )
@@
       (project "8bit_CPU-V0_1"
         (path "/81b49a11-4d6c-4532-89fe-728a8cf00278/25bbece4-880f-4fa1-94ee-76ee775f4584"
-          (reference "U13") (unit 1)
+          (reference "U9") (unit 1)
         )
       )
@@
         )
         (path "/81b49a11-4d6c-4532-89fe-728a8cf00278/25bbece4-880f-4fa1-94ee-76ee775f4584"
-          (reference "U12") (unit 1)
+          (reference "U10") (unit 1)
         )
       )
@@
         )
         (path "/81b49a11-4d6c-4532-89fe-728a8cf00278/25bbece4-880f-4fa1-94ee-76ee775f4584"
-          (reference "C12") (unit 1)
+          (reference "C10") (unit 1)
         )
       )
@@
         )
         (path "/81b49a11-4d6c-4532-89fe-728a8cf00278/25bbece4-880f-4fa1-94ee-76ee775f4584"
-          (reference "U10") (unit 1)
+          (reference "U12") (unit 1)
         )
       )
@@
         )
         (path "/81b49a11-4d6c-4532-89fe-728a8cf00278/25bbece4-880f-4fa1-94ee-76ee775f4584"
-          (reference "U9") (unit 1)
+          (reference "U27") (unit 1)
         )
       )
@@
         )
         (path "/81b49a11-4d6c-4532-89fe-728a8cf00278/25bbece4-880f-4fa1-94ee-76ee775f4584"
-          (reference "C13") (unit 1)
+          (reference "C9") (unit 1)
         )
       )
@@
   (symbol (lib_id "74xx:74LS04") (at 72.39 135.89 0) (unit 2)
     (in_bom yes) (on_board yes) (dnp no)
-    (property "Reference" "U13" (at 71.12 135.89 0)
+    (property "Reference" "U9" (at 71.12 135.89 0)
       (effects (font (size 1.27 1.27)))
     )
@@
       (project "8bit_CPU-V0_1"
         (path "/81b49a11-4d6c-4532-89fe-728a8cf00278/25bbece4-880f-4fa1-94ee-76ee775f4584"
-          (reference "U13") (unit 2)
+          (reference "U9") (unit 2)
         )
       )
@@
         )
         (path "/81b49a11-4d6c-4532-89fe-728a8cf00278/25bbece4-880f-4fa1-94ee-76ee775f4584"
-          (reference "C10") (unit 1)
-        )
-      )
+          (reference "C12") (unit 1)
+        )
+      )
