File: 8bit_CPU-V0_1/ALU2_ands.kicad_sch (KiCad schematic)
At the start: 2 parts, among them U6 74LS245

Commit message: ALU finished
Parts:
- added C1 (x3): 0.1uF, symbol Device:C
- added U21, U23, U24, U8: 74LS08, symbol 74xx:74LS08
- added U22: 74LS04, symbol 74xx:74LS04
Connections:
- net ALU2_Ain_0: now also U8.1
- net ALU2_Ain_1: now also U23.4
- net ALU2_Ain_2: now also U21.9
- net ALU2_Ain_3: now also U21.12
- net ALU2_Ain_4: now also U23.1
- net ALU2_Ain_5: now also U24.4
- net ALU2_Ain_6: now also U23.9
- net ALU2_Ain_7: now also U23.12
- net ALU2_Bin_0: now also U8.2
- net ALU2_Bin_1: now also U23.5
- net ALU2_Bin_2: now also U21.10
- net ALU2_Bin_3: now also U21.13
- net ALU2_Bin_4: now also U23.2
- net ALU2_Bin_5: now also U24.5
- net ALU2_Bin_6: now also U23.10
- net ALU2_Bin_7: now also U23.13
- net ANDS: now also U22.1
- net GND: now also C1.2, C1.2, C1.2, U22.7 (GND), U23.7 (GND), U24.7 (GND)
- net VCC: now also U6.1 (A->B), C1.1, C1.1, C1.1, U22.14 (VCC), U23.14 (VCC), U24.14 (VCC)
- net at U6.19 (CE): now also U22.2
- net at U6.2 (A0): now also U8.3
- net at U6.3 (A1): now also U23.6
- net at U6.4 (A2): now also U21.8
- net at U6.5 (A3): now also U21.11
- net at U6.6 (A4): now also U23.3
- net at U6.7 (A5): now also U24.6
- net at U6.8 (A6): now also U23.8
- net at U6.9 (A7): now also U23.11
Other:
- company: (none) -> PRP-DIY
- title: (none) -> PRP-6502 -- ALU2 : ANDS
- moved on the sheet: C6, U6

Commit message: update.
Parts:
- removed C1: 0.1uF, symbol Device:C
- removed unit 7 of U22
- renumbered U23 to U16, U24 to U16, U21 to U17, U23 to U17, U8 to U17, U24 to U17, U22 to U26
Connections:
- net ALU2_Ain_0: now also U17.9; no longer U17.1
- net ALU2_Ain_1: now also U17.12; no longer U17.4
- net ALU2_Ain_2: now also U17.4; no longer U17.9
- net ALU2_Ain_3: now also U17.1; no longer U17.12
- net ALU2_Ain_4: now also U16.9; no longer U16.1
- net ALU2_Ain_5: now also U16.12; no longer U16.4
- net ALU2_Ain_6: now also U16.4; no longer U16.9
- net ALU2_Ain_7: now also U16.1; no longer U16.12
- net ALU2_Bin_0: now also U17.10; no longer U17.2
- net ALU2_Bin_1: now also U17.13; no longer U17.5
- net ALU2_Bin_2: now also U17.5; no longer U17.10
- net ALU2_Bin_3: now also U17.2; no longer U17.13
- net ALU2_Bin_4: now also U16.10; no longer U16.2
- net ALU2_Bin_5: now also U16.13; no longer U16.5
- net ALU2_Bin_6: now also U16.5; no longer U16.10
- net ALU2_Bin_7: now also U16.2; no longer U16.13
- net ANDS: now also U26.11; no longer U26.1
- net at U6.5 (A3): now also U17.3; no longer U17.11
- net at U6.6 (A4): now also U16.8; no longer U16.3
- net at U6.8 (A6): now also U16.6; no longer U16.8
- net at U6.19 (CE): now also U26.10; no longer U26.2
- net at U6.2 (A0): now also U17.8; no longer U17.3
- net at U6.3 (A1): now also U17.11; no longer U17.6
- net at U6.4 (A2): now also U17.6; no longer U17.8
- net at U6.7 (A5): now also U16.11; no longer U16.6
- net at U6.9 (A7): now also U16.3; no longer U16.11
