File: 8bit_CPU-V0_1/ALU3_eors.kicad_sch (KiCad schematic)
At the start: 2 parts, among them U6 74LS245

Commit message: ALU finished
Parts:
- added C1 (x3): 0.1uF, symbol Device:C
- added U22: 74LS04, symbol 74xx:74LS04
- added U25, U26: 74LS86, symbol 74xx:74LS86
Connections:
- net ALU3_Ain_0: now also U25.1
- net ALU3_Ain_1: now also U25.4
- net ALU3_Ain_2: now also U25.9
- net ALU3_Ain_3: now also U25.12
- net ALU3_Ain_4: now also U26.1
- net ALU3_Ain_5: now also U26.4
- net ALU3_Ain_6: now also U26.9
- net ALU3_Ain_7: now also U26.12
- net ALU3_Bin_0: now also U25.2
- net ALU3_Bin_1: now also U25.5
- net ALU3_Bin_2: now also U25.10
- net ALU3_Bin_3: now also U25.13
- net ALU3_Bin_4: now also U26.2
- net ALU3_Bin_5: now also U26.5
- net ALU3_Bin_6: now also U26.10
- net ALU3_Bin_7: now also U26.13
- net EORS: now also U22.1
- net GND: now also C1.2, C1.2, C1.2, U22.7 (GND), U25.7 (GND), U26.7 (GND)
- net VCC: now also U6.1 (A->B), C1.1, C1.1, C1.1, U22.14 (VCC), U25.14 (VCC), U26.14 (VCC)
- net at U6.19 (CE): now also U22.2
- net at U6.2 (A0): now also U25.3
- net at U6.3 (A1): now also U25.6
- net at U6.4 (A2): now also U25.8
- net at U6.5 (A3): now also U25.11
- net at U6.6 (A4): now also U26.3
- net at U6.7 (A5): now also U26.6
- net at U6.8 (A6): now also U26.8
- net at U6.9 (A7): now also U26.11
Other:
- company: (none) -> PRP-DIY
- title: (none) -> PRP-6502 -- ALU3 : EORS

Commit message: update.
Parts:
- removed C1: 0.1uF, symbol Device:C
- removed unit 7 of U22
- renumbered U26 to U19, U25 to U20
Connections:
- net ALU3_Ain_0: now also U20.9; no longer U20.1
- net ALU3_Ain_1: now also U20.12; no longer U20.4
- net ALU3_Ain_2: now also U20.4; no longer U20.9
- net ALU3_Ain_3: now also U20.1; no longer U20.12
- net ALU3_Ain_4: now also U19.9; no longer U19.1
- net ALU3_Ain_5: now also U19.12; no longer U19.4
- net ALU3_Ain_6: now also U19.4; no longer U19.9
- net ALU3_Ain_7: now also U19.1; no longer U19.12
- net ALU3_Bin_0: now also U20.10; no longer U20.2
- net ALU3_Bin_1: now also U20.13; no longer U20.5
- net ALU3_Bin_2: now also U20.5; no longer U20.10
- net ALU3_Bin_3: now also U20.2; no longer U20.13
- net ALU3_Bin_4: now also U19.10; no longer U19.2
- net ALU3_Bin_5: now also U19.13; no longer U19.5
- net ALU3_Bin_6: now also U19.5; no longer U19.10
- net ALU3_Bin_7: now also U19.2; no longer U19.13
- net at U6.6 (A4): now also U19.8; no longer U19.3
- net at U6.8 (A6): now also U19.6; no longer U19.8
- net at U6.2 (A0): now also U20.8; no longer U20.3
- net at U6.3 (A1): now also U20.11; no longer U20.6
- net at U6.4 (A2): now also U20.6; no longer U20.8
- net at U6.5 (A3): now also U20.3; no longer U20.11
- net at U6.7 (A5): now also U19.11; no longer U19.6
- net at U6.9 (A7): now also U19.3; no longer U19.11
