File: 8bit_CPU-V0_1/ALU4_ors.kicad_sch (KiCad schematic)
At the start: 10 parts, among them U17 74LS32, U22 74LS04, U29 74LS32, U30 74LS32, U6 74LS245, U9 74LS32

Commit message: update.
Parts:
- removed C1: 0.1uF, symbol Device:C
- removed unit 7 of U22
- renumbered U30 to U22, U29 to U22, U9 to U23, U29 to U23, U17 to U23
Connections:
- net ALU4_Ain_0: now also U23.9; no longer U23.1
- net ALU4_Ain_1: now also U23.12; no longer U23.4
- net ALU4_Ain_2: now also U23.4; no longer U23.9
- net ALU4_Ain_3: now also U23.1; no longer U23.12
- net ALU4_Ain_4: now also U22.9; no longer U22.1
- net ALU4_Ain_5: now also U22.12; no longer U22.4
- net ALU4_Ain_6: now also U22.4; no longer U22.9
- net ALU4_Ain_7: now also U22.1; no longer U22.12
- net ALU4_Bin_0: now also U23.10; no longer U23.2
- net ALU4_Bin_1: now also U23.13; no longer U23.5
- net ALU4_Bin_2: now also U23.5; no longer U23.10
- net ALU4_Bin_3: now also U23.2; no longer U23.13
- net ALU4_Bin_4: now also U22.10; no longer U22.2
- net ALU4_Bin_5: now also U22.13; no longer U22.5
- net ALU4_Bin_6: now also U22.5; no longer U22.10
- net ALU4_Bin_7: now also U22.2; no longer U22.13
- net at U6.7 (A5): now also U22.11; no longer U22.6
- net at U6.4 (A2): now also U23.6; no longer U23.8
- net at U6.3 (A1): now also U23.11; no longer U23.6
- net at U6.9 (A7): now also U22.3; no longer U22.11
- net at U6.2 (A0): now also U23.8; no longer U23.3
- net at U6.5 (A3): now also U23.3; no longer U23.11
- net at U6.6 (A4): now also U22.8; no longer U22.3
- net at U6.8 (A6): now also U22.6; no longer U22.8
