File: 8bit_CPU-V0_1/ALU5_srs.kicad_sch (KiCad schematic)
At the start: 7 parts, among them U22 74LS04, U24 74LS08, U38 74LS08, U40 74LS86, U6 74LS245

Commit message: ALU finished
Changed lines of the file:
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@@
   )
   (symbol (lib_id "74xx:74LS86") (at 242.57 48.26 0) (unit 1)
-    (in_bom yes) (on_board yes) (dnp no) (fields_autoplaced)
-    (property "Reference" "U40" (at 242.2652 39.37 0)
+    (in_bom yes) (on_board yes) (dnp no)
+    (property "Reference" "U40" (at 242.2735 48.26 0)
       (effects (font (size 1.27 1.27)))
     )
     (property "Value" "74LS86" (at 242.2652 41.91 0)
-      (effects (font (size 1.27 1.27)))
+      (effects (font (size 1.27 1.27)) hide)
     )
     (property "Footprint" "" (at 242.57 48.26 0)
@@
   )
   (symbol (lib_id "74xx:74LS08") (at 191.77 40.64 0) (unit 1)
-    (in_bom yes) (on_board yes) (dnp no) (fields_autoplaced)
-    (property "Reference" "U24" (at 191.7617 31.75 0)
+    (in_bom yes) (on_board yes) (dnp no)
+    (property "Reference" "U24" (at 191.77 40.64 0)
       (effects (font (size 1.27 1.27)))
     )
     (property "Value" "74LS08" (at 191.7617 34.29 0)
-      (effects (font (size 1.27 1.27)))
+      (effects (font (size 1.27 1.27)) hide)
     )
     (property "Footprint" "" (at 191.77 40.64 0)
@@
   )
   (symbol (lib_id "74xx:74LS08") (at 217.17 57.15 0) (unit 2)
-    (in_bom yes) (on_board yes) (dnp no) (fields_autoplaced)
-    (property "Reference" "U38" (at 217.1617 48.26 0)
+    (in_bom yes) (on_board yes) (dnp no)
+    (property "Reference" "U38" (at 217.17 57.15 0)
       (effects (font (size 1.27 1.27)))
     )
     (property "Value" "74LS08" (at 217.1617 50.8 0)
-      (effects (font (size 1.27 1.27)))
+      (effects (font (size 1.27 1.27)) hide)
     )
     (property "Footprint" "" (at 217.17 57.15 0)

Commit message: Refining schematics
Parts:
- added D5: LED, symbol Device:LED
- added R1: 330, symbol Device:R_US
Connections:
- net ACR: now also D5.2 (A)
- net GND: now also R1.2
- new net: D5.1 (K), R1.1
Changed lines of the file:
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@@
   (junction (at 201.93 78.74) (diameter 0) (color 0 0 0 0)
   )
+  (junction (at 255.27 48.26) (diameter 0) (color 0 0 0 0)
+  )
   (junction (at 220.98 87.63) (diameter 0) (color 0 0 0 0)
   )
@@
     (stroke (width 0) (type default))
   )
+  (wire (pts (xy 271.78 60.96) (xy 267.97 60.96))
+    (stroke (width 0) (type default))
+  )
   (wire (pts (xy 233.68 87.63) (xy 237.49 87.63))
     (stroke (width 0) (type default))
@@
     (stroke (width 0) (type default))
   )
+  (wire (pts (xy 260.35 60.96) (xy 255.27 60.96))
+    (stroke (width 0) (type default))
+  )
   (wire (pts (xy 50.8 85.09) (xy 139.7 85.09))
     (stroke (width 0) (type default))
@@
     (stroke (width 0) (type default))
   )
+  (wire (pts (xy 255.27 48.26) (xy 255.27 50.8))
+    (stroke (width 0) (type default))
+  )
   (wire (pts (xy 144.78 97.79) (xy 208.28 97.79))
     (stroke (width 0) (type default))
@@
     (stroke (width 0) (type default))
   )
+  (wire (pts (xy 255.27 60.96) (xy 255.27 58.42))
+    (stroke (width 0) (type default))
+  )
   (wire (pts (xy 233.68 110.49) (xy 242.57 110.49))
     (stroke (width 0) (type default))
@@
   )
   (wire (pts (xy 255.27 48.26) (xy 255.27 45.72))
+    (stroke (width 0) (type default))
+  )
+  (wire (pts (xy 271.78 63.5) (xy 271.78 60.96))
     (stroke (width 0) (type default))
   )
@@
         (path "/81b49a11-4d6c-4532-89fe-728a8cf00278/5c82f420-9238-4483-85b4-9976015269a2"
           (reference "#PWR095") (unit 1)
+        )
+      )
+    )
+  )
+  (symbol (lib_id "Device:R_US") (at 264.16 60.96 90) (unit 1)
+    (in_bom yes) (on_board yes) (dnp no) (fields_autoplaced)
+    (property "Reference" "R1" (at 264.16 54.61 90)
+      (effects (font (size 1.27 1.27)))
+    )
+    (property "Value" "330" (at 264.16 57.15 90)
+      (effects (font (size 1.27 1.27)))
+    )
+    (property "Footprint" "" (at 264.414 59.944 90)
+      (effects (font (size 1.27 1.27)) hide)
+    )
+    (property "Datasheet" "~" (at 264.16 60.96 0)
+      (effects (font (size 1.27 1.27)) hide)
+    )
+    (pin "1")
+    (pin "2")
+    (instances
+      (project "8bit_CPU-V0_1"
+        (path "/81b49a11-4d6c-4532-89fe-728a8cf00278/5c82f420-9238-4483-85b4-9976015269a2"
+          (reference "R1") (unit 1)
+        )
+      )
+    )
+  )
+  (symbol (lib_id "Device:LED") (at 255.27 54.61 90) (unit 1)
+    (in_bom yes) (on_board yes) (dnp no)
+    (property "Reference" "D5" (at 256.54 52.07 90)
+      (effects (font (size 1.27 1.27)) (justify right))
+    )
+    (property "Value" "LED" (at 251.46 56.1975 0)
+      (effects (font (size 1.27 1.27)) hide)
+    )
+    (property "Footprint" "" (at 255.27 54.61 0)
+      (effects (font (size 1.27 1.27)) hide)
+    )
+    (property "Datasheet" "~" (at 255.27 54.61 0)
+      (effects (font (size 1.27 1.27)) hide)
+    )
+    (pin "1")
+    (pin "2")
+    (instances
+      (project "8bit_CPU-V0_1"
+        (path "/81b49a11-4d6c-4532-89fe-728a8cf00278/35c1fb24-0486-4fe0-9b7f-61a5bd7cfd0a"
+          (reference "D5") (unit 1)
+        )
+        (path "/81b49a11-4d6c-4532-89fe-728a8cf00278/61dc0d7a-8fde-4fbd-b542-ed8316c8cea0"
+          (reference "D21") (unit 1)
+        )
+        (path "/81b49a11-4d6c-4532-89fe-728a8cf00278/5c82f420-9238-4483-85b4-9976015269a2"
+          (reference "D25") (unit 1)
         )
       )
@@
         )
       )
+    )
+  )
+  (symbol (lib_id "power:GND") (at 271.78 63.5 0) (unit 1)
+    (in_bom yes) (on_board yes) (dnp no)
+    (property "Reference" "#PWR017" (at 271.78 69.85 0)
+      (effects (font (size 1.27 1.27)) hide)
+    )
+    (property "Value" "GND" (at 271.78 67.31 0)
+      (effects (font (size 1.27 1.27)))
+    )
+    (property "Footprint" "" (at 271.78 63.5 0)
+      (effects (font (size 1.27 1.27)) hide)
+    )
+    (property "Datasheet" "" (at 271.78 63.5 0)
+      (effects (font (size 1.27 1.27)) hide)
+    )
+    (pin "1")
+    (instances
+      (project "8bit_CPU-V0_1"
+        (path "/81b49a11-4d6c-4532-89fe-728a8cf00278/35c1fb24-0486-4fe0-9b7f-61a5bd7cfd0a"
+          (reference "#PWR017") (unit 1)
+        )
+        (path "/81b49a11-4d6c-4532-89fe-728a8cf00278/2506dba5-d3a6-49a3-9eb6-4c25813b2799"
+          (reference "#PWR044") (unit 1)
+        )
+        (path "/81b49a11-4d6c-4532-89fe-728a8cf00278/ced47c2c-41ac-49d8-adf8-5e05670f7615"
+          (reference "#PWR065") (unit 1)
+        )
+        (path "/81b49a11-4d6c-4532-89fe-728a8cf00278/7f9f7569-f610-4381-81c7-c45e5846f6ba"
+          (reference "#PWR077") (unit 1)
+        )
+        (path "/81b49a11-4d6c-4532-89fe-728a8cf00278/eed8f768-7506-4df5-b01f-6a23e528aa72"
+          (reference "#PWR089") (unit 1)
+        )
+        (path "/81b49a11-4d6c-4532-89fe-728a8cf00278/5c82f420-9238-4483-85b4-9976015269a2"
+          (reference "#PWR0107") (unit 1)
+        )
+      )

Commit message: update.
Parts:
- removed U22: 74LS04, symbol 74xx:74LS04
- added unit 5 of U42
- added unit 5 of U43
- renumbered U24 to U42, U38 to U42, U40 to U43
Connections:
- net ACR: now also U43.6; no longer U43.3
- net ALU5_Ain_0: now also U42.12; no longer U42.4
- net SRS: now also U42.13; no longer U42.5
- net SUMS_CARRY(ALU1): now also U42.9; no longer U42.1
- net at U22.2, U6.19 (CE): now also U42.10
- new net: U42.8, U43.4
- new net: U42.11, U43.5
Other:
- moved on the sheet: U22A
