File: 8bit_CPU-V0_1/ALU5_srs.kicad_sch (KiCad schematic)
At the start: 9 parts, among them U22 74LS04, U24 74LS08, U38 74LS08, U40 74LS86, U6 74LS245

Commit message: New update
Parts:
- removed U22: 74LS04, symbol 74xx:74LS04
- added C1 (x2): 0.1uF, symbol Device:C
- added unit 5 of U42
- added unit 5 of U43
- renumbered U24 to U42, U38 to U42, U40 to U43
Connections:
- net ACR: now also U43.6; no longer U43.3
- net ALU5_Ain_0: now also U42.12; no longer U42.4
- net GND: now also C1.2, C1.2, U42.7 (GND), U43.7 (GND)
- net SRS: now also U42.13; no longer U42.5
- net SUMS_CARRY(ALU1): now also U42.9; no longer U42.1
- net VCC: now also C1.1, C1.1, U42.14 (VCC), U43.14 (VCC)
- net at U22.2, U6.19 (CE): now also U42.10
- new net: U42.8, U43.4
- new net: U42.11, U43.5
Other:
- moved on the sheet: U22A
