File: 8bit_CPU-V0_1/BInput_reg.kicad_sch (KiCad schematic)
At the start: 27 parts, among them U1 74LS86, U2 74LS86, U3 74LS173, U4 74LS173, U5 74HCT04, U6 74LS245, U7 74LS245, U8 74LS08, U9 74LS32

Commit message: ALU finished
Parts:
- renumbered C6 to C1, C7 to C2, C2 to C3, C1 to C4, C3 to C5, C4 to C6, C5 to C7, U6 to U1, U7 to U2, U2 to U3, U1 to U4, U3 to U5, U4 to U6, U5 to U7
Connections:
- net ADL/ADD: now also U7.9; no longer U7.5
- net DB/ADD: now also U9.12; no longer U9.1
- net ~{Bin_RST}: now also U7.9; no longer U7.1
- net ~{DB}/ADD: now also U3.10, U3.13, U3.2, U3.5, U4.10, U4.13, U4.2, U4.5, U9.13; no longer U3.10, U3.13, U3.2, U3.5, U4.10, U4.13, U4.2, U4.5, U9.2
- net at U1.18 (B0), U2.18 (B0): now also U4.9; no longer U4.1
- net at U5.14 (D0): now also U4.8; no longer U4.3
- net at U5.10 (E2), U5.9 (E1), U6.10 (E2)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: now also U8.8; no longer U8.3
- net at U5.11 (D3): now also U4.3; no longer U4.11
- net at U5.12 (D2): now also U4.6; no longer U4.8
- net at U5.13 (D1): now also U4.11; no longer U4.6
- net at U5.15 (Mr), U6.15 (Mr): now also U7.8; no longer U7.2
- net at U6.12 (D2): now also U3.6; no longer U3.8
- net at U1.12 (B6), U2.12 (B6): now also U3.4; no longer U3.9
- net at U1.11 (B7), U2.11 (B7): now also U3.1; no longer U3.12
- net at U1.13 (B5), U2.13 (B5): now also U3.12; no longer U3.4
- net at U1.14 (B4), U2.14 (B4): now also U3.9; no longer U3.1
- net at U1.15 (B3), U2.15 (B3): now also U4.1; no longer U4.12
- net at U1.16 (B2), U2.16 (B2): now also U4.4; no longer U4.9
- net at U1.17 (B1), U2.17 (B1): now also U4.12; no longer U4.4
- net at U6.11 (D3): now also U3.3; no longer U3.11
- net at U6.13 (D1): now also U3.11; no longer U3.6
- net at U6.14 (D0): now also U3.8; no longer U3.3
- new net: U1.19 (CE), U7.12, U8.10
- new net: U7.13, U9.11
- new net: U2.19 (CE), U7.8, U8.9
Other:
- note added: "24 AWG"
- note added: "Test Switch #1"
- note added: "Test Switch #2"
- note added: "Test Switch #3"
- company: (none) -> PRP-DIY
- title: (none) -> PRP-6502 -- ALU : B Input Register
- moved on the sheet: U7F

Commit message: update.
Parts:
- renumbered C8 to C27, C7 to C5, C9 to C6, C6 to C7, C5 to C8, U9 to U27, U7 to U5, U8 to U6, U6 to U7, U5 to U8
Connections:
- net ~{Bin_RST}: now also U5.11; no longer U5.9
- net at U7.15 (Mr), U8.15 (Mr): now also U5.10; no longer U5.8
Changed lines of the file:
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@@
   (title_block
     (title "PRP-6502 -- ALU : B Input Register")
-    (date "2023-07-02")
-    (rev "0")
+    (date "2023-07-06")
+    (rev "1")
     (company "PRP-DIY")
   )
@@
   )
   (wire (pts (xy 182.88 109.22) (xy 182.88 106.68))
-    (stroke (width 0) (type default))
-  )
-  (wire (pts (xy 63.5 62.23) (xy 67.31 62.23))
     (stroke (width 0) (type default))
   )
@@
   (symbol (lib_id "Device:C") (at 208.28 24.13 90) (unit 1)
     (in_bom yes) (on_board yes) (dnp no)
-    (property "Reference" "C5" (at 209.55 20.32 90)
+    (property "Reference" "C8" (at 209.55 20.32 90)
       (effects (font (size 1.27 1.27)) (justify left))
     )
@@
       (project "8bit_CPU-V0_1"
         (path "/81b49a11-4d6c-4532-89fe-728a8cf00278/35c1fb24-0486-4fe0-9b7f-61a5bd7cfd0a"
-          (reference "C5") (unit 1)
+          (reference "C8") (unit 1)
         )
       )
@@
   (symbol (lib_id "74xx:74LS08") (at 60.96 179.07 0) (unit 5)
     (in_bom yes) (on_board yes) (dnp no) (fields_autoplaced)
-    (property "Reference" "U8" (at 67.31 177.8 0)
+    (property "Reference" "U6" (at 67.31 177.8 0)
       (effects (font (size 1.27 1.27)) (justify left))
     )
@@
       (project "8bit_CPU-V0_1"
         (path "/81b49a11-4d6c-4532-89fe-728a8cf00278/35c1fb24-0486-4fe0-9b7f-61a5bd7cfd0a"
-          (reference "U8") (unit 5)
+          (reference "U6") (unit 5)
         )
       )
@@
   (symbol (lib_id "74xx:74LS32") (at 27.94 177.8 0) (unit 5)
     (in_bom yes) (on_board yes) (dnp no) (fields_autoplaced)
-    (property "Reference" "U9" (at 34.29 176.53 0)
+    (property "Reference" "U27" (at 34.29 176.53 0)
       (effects (font (size 1.27 1.27)) (justify left))
     )
@@
       (project "8bit_CPU-V0_1"
         (path "/81b49a11-4d6c-4532-89fe-728a8cf00278/35c1fb24-0486-4fe0-9b7f-61a5bd7cfd0a"
-          (reference "U9") (unit 5)
+          (reference "U27") (unit 5)
         )
       )
@@
   (symbol (lib_id "74xx:74LS173") (at 199.39 52.07 0) (unit 1)
     (in_bom yes) (on_board yes) (dnp no)
-    (property "Reference" "U5" (at 193.04 33.02 0)
+    (property "Reference" "U8" (at 193.04 33.02 0)
       (effects (font (size 1.27 1.27)) (justify left))
     )
@@
       (project "8bit_CPU-V0_1"
         (path "/81b49a11-4d6c-4532-89fe-728a8cf00278/35c1fb24-0486-4fe0-9b7f-61a5bd7cfd0a"
-          (reference "U5") (unit 1)
-        )
-      )
-    )
-  )
-  (symbol (lib_id "74xx:74HCT04") (at 63.5 156.21 0) (unit 4)
-    (in_bom yes) (on_board yes) (dnp no)
-    (property "Reference" "U7" (at 62.23 156.21 0)
+          (reference "U8") (unit 1)
+        )
+      )
+    )
+  )
+  (symbol (lib_id "74xx:74HCT04") (at 63.5 156.21 0) (unit 5)
+    (in_bom yes) (on_board yes) (dnp no)
+    (property "Reference" "U5" (at 62.23 156.21 0)
       (effects (font (size 1.27 1.27)))
     )
@@
       (project "8bit_CPU-V0_1"
         (path "/81b49a11-4d6c-4532-89fe-728a8cf00278/35c1fb24-0486-4fe0-9b7f-61a5bd7cfd0a"
-          (reference "U7") (unit 4)
+          (reference "U5") (unit 5)
         )
       )
@@
   (symbol (lib_id "Device:C") (at 52.07 179.07 0) (unit 1)
     (in_bom yes) (on_board yes) (dnp no)
-    (property "Reference" "C8" (at 46.99 176.53 0)
+    (property "Reference" "C27" (at 46.99 176.53 0)
       (effects (font (size 1.27 1.27)) (justify left))
     )
@@
       (project "8bit_CPU-V0_1"
         (path "/81b49a11-4d6c-4532-89fe-728a8cf00278/35c1fb24-0486-4fe0-9b7f-61a5bd7cfd0a"
-          (reference "C8") (unit 1)
+          (reference "C27") (unit 1)
         )
       )
@@
     )
   )
-  (symbol (lib_id "power:GND") (at 63.5 62.23 0) (unit 1)
-    (in_bom yes) (on_board yes) (dnp no)
-    (property "Reference" "#PWR021" (at 63.5 68.58 0)
-      (effects (font (size 1.27 1.27)) hide)
-    )
-    (property "Value" "GND" (at 63.5 66.04 0)
-      (effects (font (size 1.27 1.27)))
-    )
-    (property "Footprint" "" (at 63.5 62.23 0)
-      (effects (font (size 1.27 1.27)) hide)
-    )
-    (property "Datasheet" "" (at 63.5 62.23 0)
+  (symbol (lib_id "power:GND") (at 67.31 62.23 0) (unit 1)
+    (in_bom yes) (on_board yes) (dnp no)
+    (property "Reference" "#PWR021" (at 67.31 68.58 0)
+      (effects (font (size 1.27 1.27)) hide)
+    )
+    (property "Value" "GND" (at 67.31 66.04 0)
+      (effects (font (size 1.27 1.27)))
+    )
+    (property "Footprint" "" (at 67.31 62.23 0)
+      (effects (font (size 1.27 1.27)) hide)
+    )
+    (property "Datasheet" "" (at 67.31 62.23 0)
       (effects (font (size 1.27 1.27)) hide)
     )
@@
   (symbol (lib_id "74xx:74LS173") (at 199.39 111.76 0) (unit 1)
     (in_bom yes) (on_board yes) (dnp no)
-    (property "Reference" "U6" (at 194.31 92.71 0)
+    (property "Reference" "U7" (at 194.31 92.71 0)
       (effects (font (size 1.27 1.27)))
     )
@@
       (project "8bit_CPU-V0_1"
         (path "/81b49a11-4d6c-4532-89fe-728a8cf00278/35c1fb24-0486-4fe0-9b7f-61a5bd7cfd0a"
-          (reference "U6") (unit 1)
+          (reference "U7") (unit 1)
         )
       )
@@
   (symbol (lib_id "74xx:74HCT04") (at 92.71 177.8 0) (unit 7)
     (in_bom yes) (on_board yes) (dnp no) (fields_autoplaced)
-    (property "Reference" "U7" (at 99.06 176.53 0)
+    (property "Reference" "U5" (at 99.06 176.53 0)
       (effects (font (size 1.27 1.27)) (justify left))
     )
@@
       (project "8bit_CPU-V0_1"
         (path "/81b49a11-4d6c-4532-89fe-728a8cf00278/35c1fb24-0486-4fe0-9b7f-61a5bd7cfd0a"
-          (reference "U7") (unit 7)
+          (reference "U5") (unit 7)
         )
       )
@@
   (symbol (lib_id "Device:C") (at 83.82 177.8 0) (unit 1)
     (in_bom yes) (on_board yes) (dnp no)
-    (property "Reference" "C7" (at 78.74 175.26 0)
+    (property "Reference" "C5" (at 78.74 175.26 0)
       (effects (font (size 1.27 1.27)) (justify left))
     )
@@
       (project "8bit_CPU-V0_1"
         (path "/81b49a11-4d6c-4532-89fe-728a8cf00278/35c1fb24-0486-4fe0-9b7f-61a5bd7cfd0a"
-          (reference "C7") (unit 1)
+          (reference "C5") (unit 1)
         )
       )
@@
   (symbol (lib_id "74xx:74LS32") (at 35.56 138.43 0) (unit 4)
     (in_bom yes) (on_board yes) (dnp no)
-    (property "Reference" "U9" (at 35.56 138.43 0)
+    (property "Reference" "U27" (at 35.56 138.43 0)
       (effects (font (size 1.27 1.27)))
     )
@@
       (project "8bit_CPU-V0_1"
         (path "/81b49a11-4d6c-4532-89fe-728a8cf00278/35c1fb24-0486-4fe0-9b7f-61a5bd7cfd0a"
-          (reference "U9") (unit 4)
+          (reference "U27") (unit 4)
         )
       )
@@
   (symbol (lib_id "Device:C") (at 215.9 85.09 270) (unit 1)
     (in_bom yes) (on_board yes) (dnp no)
-    (property "Reference" "C6" (at 214.63 81.28 90)
+    (property "Reference" "C7" (at 214.63 81.28 90)
       (effects (font (size 1.27 1.27)) (justify left))
     )
@@
       (project "8bit_CPU-V0_1"
         (path "/81b49a11-4d6c-4532-89fe-728a8cf00278/35c1fb24-0486-4fe0-9b7f-61a5bd7cfd0a"
-          (reference "C6") (unit 1)
+          (reference "C7") (unit 1)
         )
       )
@@
   (symbol (lib_id "74xx:74LS08") (at 107.95 129.54 0) (unit 3)
     (in_bom yes) (on_board yes) (dnp no)
-    (property "Reference" "U8" (at 107.95 129.54 0)
+    (property "Reference" "U6" (at 107.95 129.54 0)
       (effects (font (size 1.27 1.27)))
     )
@@
       (project "8bit_CPU-V0_1"
         (path "/81b49a11-4d6c-4532-89fe-728a8cf00278/35c1fb24-0486-4fe0-9b7f-61a5bd7cfd0a"
-          (reference "U8") (unit 3)
+          (reference "U6") (unit 3)
         )
       )
@@
   (symbol (lib_id "74xx:74HCT04") (at 53.34 138.43 0) (unit 6)
     (in_bom yes) (on_board yes) (dnp no)
-    (property "Reference" "U7" (at 52.07 138.43 0)
+    (property "Reference" "U5" (at 52.07 138.43 0)
       (effects (font (size 1.27 1.27)))
     )
@@
       (project "8bit_CPU-V0_1"
         (path "/81b49a11-4d6c-4532-89fe-728a8cf00278/35c1fb24-0486-4fe0-9b7f-61a5bd7cfd0a"
-          (reference "U7") (unit 6)
+          (reference "U5") (unit 6)
         )
       )
@@
   (symbol (lib_id "Device:C") (at 19.05 177.8 0) (unit 1)
     (in_bom yes) (on_board yes) (dnp no)
-    (property "Reference" "C9" (at 13.97 175.26 0)
+    (property "Reference" "C6" (at 13.97 175.26 0)
       (effects (font (size 1.27 1.27)) (justify left))
     )
@@
       (project "8bit_CPU-V0_1"
         (path "/81b49a11-4d6c-4532-89fe-728a8cf00278/35c1fb24-0486-4fe0-9b7f-61a5bd7cfd0a"
-          (reference "C9") (unit 1)
+          (reference "C6") (unit 1)
         )
       )
@@
   (symbol (lib_id "74xx:74HCT04") (at 40.64 121.92 0) (unit 4)
     (in_bom yes) (on_board yes) (dnp no)
-    (property "Reference" "U7" (at 39.37 121.92 0)
+    (property "Reference" "U5" (at 39.37 121.92 0)
       (effects (font (size 1.27 1.27)))
     )
@@
       (project "8bit_CPU-V0_1"
         (path "/81b49a11-4d6c-4532-89fe-728a8cf00278/35c1fb24-0486-4fe0-9b7f-61a5bd7cfd0a"
-          (reference "U7") (unit 4)
-        )
-      )
+          (reference "U5") (unit 4)
+        )
+      )
