File: 8bit_CPU-V0_1/8bit_CPU-V0_1.kicad_sch (KiCad schematic)
At the start: 0 parts

Commit message: New update
Other:
- added sheet Accumulator (AC) (Accumulator.kicad_sch)
- added sheet Clock Generator (CLK_gen.kicad_sch)
- added sheet Decimal adjuster Adders (Decimal adjustet.kicad_sch)
- added sheet Overflow dectection (OVR_det.kicad_sch)
- added sheet Processor Status Register (P) (Stat_reg.kicad_sch)
- added sheet Program Counter Low (PCL & PCLS) (PCL.kicad_sch)
- added sheet Stack Pointer (S) (Stack_Pointer.kicad_sch)
- added sheet X Register (X_reg.kicad_sch)
- added sheet Y Register (Y_reg.kicad_sch)
- sheet ALU1-SUMS ports: added AVR_SUMS_OUT; removed none
