File: 8bit_CPU-V0_1/8bit_CPU-V0_1.kicad_sch (KiCad schematic)
At the start: 0 parts

Commit message: Update
Other:
- added sheet Address Bus High Register (ABH) (ABH.kicad_sch)
- added sheet Address Bus Low Register (ABL) (ABL.kicad_sch)
- added sheet Input Data Latch (DL) (Data_Latch_DL.kicad_sch)
- added sheet Program Counter High (PCH & PCHS) (PCH.kicad_sch)
Changed lines of the file:
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@@
+    )
+  )
+  (sheet (at 307.34 60.96) (size 22.86 48.26) (fields_autoplaced)
+    (stroke (width 0.1524) (type solid))
+    (fill (color 0 0 0 0.0000))
+    (property "Sheetname" "Address Bus Low Register (ABL)" (at 307.34 60.2484 0)
+      (effects (font (size 1.27 1.27)) (justify left bottom))
+    )
+    (property "Sheetfile" "ABL.kicad_sch" (at 307.34 109.8046 0)
+      (effects (font (size 1.27 1.27)) (justify left top))
+    )
+    (instances
+      (project "8bit_CPU-V0_1"
+        (path "/81b49a11-4d6c-4532-89fe-728a8cf00278" (page "19"))
+      )
     )
   )
@@
     )
   )
+  (sheet (at -30.48 -144.78) (size 64.77 58.42) (fields_autoplaced)
+    (stroke (width 0.1524) (type solid))
+    (fill (color 0 0 0 0.0000))
+    (property "Sheetname" "Program Counter High (PCH & PCHS)" (at -30.48 -145.4916 0)
+      (effects (font (size 1.27 1.27)) (justify left bottom))
+    )
+    (property "Sheetfile" "PCH.kicad_sch" (at -30.48 -85.7754 0)
+      (effects (font (size 1.27 1.27)) (justify left top))
+    )
+    (instances
+      (project "8bit_CPU-V0_1"
+        (path "/81b49a11-4d6c-4532-89fe-728a8cf00278" (page "21"))
+      )
+    )
+  )
   (sheet (at 133.35 185.42) (size 43.18 52.07) (fields_autoplaced)
     (stroke (width 0.1524) (type solid))
@@
     )
   )
+  (sheet (at 386.08 82.55) (size 31.75 39.37) (fields_autoplaced)
+    (stroke (width 0.1524) (type solid))
+    (fill (color 0 0 0 0.0000))
+    (property "Sheetname" "Address Bus High Register (ABH)" (at 386.08 81.8384 0)
+      (effects (font (size 1.27 1.27)) (justify left bottom))
+    )
+    (property "Sheetfile" "ABH.kicad_sch" (at 386.08 122.5046 0)
+      (effects (font (size 1.27 1.27)) (justify left top))
+    )
+    (instances
+      (project "8bit_CPU-V0_1"
+        (path "/81b49a11-4d6c-4532-89fe-728a8cf00278" (page "20"))
+      )
+    )
+  )
   (sheet (at 306.07 127) (size 27.94 39.37) (fields_autoplaced)
     (stroke (width 0.1524) (type solid))
@@
       )
     )
+  )
+  (sheet (at 166.37 -165.1) (size 62.23 29.21) (fields_autoplaced)
+    (stroke (width 0.1524) (type solid))
+    (fill (color 0 0 0 0.0000))
+    (property "Sheetname" "Input Data Latch (DL)" (at 166.37 -165.8116 0)
+      (effects (font (size 1.27 1.27)) (justify left bottom))
+    )
+    (property "Sheetfile" "Data_Latch_DL.kicad_sch" (at 166.37 -135.3054 0)
+      (effects (font (size 1.27 1.27)) (justify left top))
+    )
+    (instances
+      (project "8bit_CPU-V0_1"
+        (path "/81b49a11-4d6c-4532-89fe-728a8cf00278" (page "22"))
+      )
+    )
