File: 8bit_CPU-V0_1/Accumulator.kicad_sch (KiCad schematic)
At the start: 7 parts, among them U41 74LS574, U56 74LS04, U6 74LS245

Commit message: Update
Changed lines of the file:
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@@
-    (effects (font (size 1.27 1.27)) (justify right))
-  )
-  (hierarchical_label "CLK" (shape input) (at 34.29 82.55 180) (fields_autoplaced)
     (effects (font (size 1.27 1.27)) (justify right))
   )
