File: 8bit_CPU-V0_1/Decimal adjustet.kicad_sch (KiCad schematic)
At the start: 12 parts, among them U51 74LS283, U52 74LS283, U53 74LS32, U54 74LS08, U55 74LS08, U56 74LS04

Commit message: Update
Changed lines of the file:
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@@
     (effects (font (size 1.27 1.27)) (justify right))
-  )
-  (hierarchical_label "CLK" (shape input) (at 26.67 143.51 0) (fields_autoplaced)
-    (effects (font (size 1.27 1.27)) (justify left))
   )
   (hierarchical_label "Decimal_AC_6" (shape output) (at 242.57 77.47 0) (fields_autoplaced)
