File: 8bit_CPU-V0_1/PCL.kicad_sch (KiCad schematic)
At the start: 11 parts, among them U50 74LS04, U54 74LS32, U56 74LS04, U61 74LS04, U62 74LS161, U63 74LS161, U64 74LS574, U65 74LS245, U66 74LS245, U67 74LS04, U68 74LS245

Commit message: Update
Parts:
- added C1 (x2), C6 (x6): 0.1uF, symbol Device:C
- added U26: 74LS04, symbol 74xx:74LS04
- added U53: 74LS32, symbol 74xx:74LS32
- added unit 2 of U70
- renumbered U68 to U63, U62 to U64, U63 to U65, U64 to U66, U65 to U67, U66 to U68, U56 to U69, U67 to U69, U61 to U69, U50 to U69, U54 to U70
Connections:
- net ADL/PCL: now also U69.5; no longer U69.3
- net GND: now also U63.10 (GND), U64.8 (GND), U65.8 (GND), U67.10 (GND), U68.10 (GND), C1.2, C1.2, C6.2, C6.2, C6.2, C6.2, C6.2, C6.2, U26.7 (GND), U53.7 (GND)
- net I/PC: now also U70.4
- net PCL/ADL: now also U69.3; no longer U69.1
- net PCL/DB: now also U69.1; no longer U69.3
- net VCC: now also U63.20 (VCC), U64.1 (~{MR}), U64.16 (VCC), U65.1 (~{MR}), U65.16 (VCC), U66.20 (VCC), U67.20 (VCC), U68.20 (VCC), C1.1, C1.1, C6.1, C6.1, C6.1, C6.1, C6.1, C6.1, U26.14 (VCC), U53.14 (VCC)
- net at U63.19 (CE): now also U69.6; no longer U69.4
- net at U67.19 (CE): now also U69.2; no longer U69.4
- net at U70.3: now also U69.9, U70.5; no longer U69.3
- net at U68.19 (CE): now also U69.4; no longer U69.2
- net at U64.9 (~{PE}), U65.9 (~{PE}): now also U69.8; no longer U69.4
- net at U64.2 (CP): now also U70.6
- net PCL_CLK renamed PCL_CLK2
Other:
- title: (none) -> Program Counter Low (PCL & PCLS)
- moved on the sheet: U64, U65
