File: 8bit_CPU-V0_1/Stack_Pointer.kicad_sch (KiCad schematic)
At the start: 19 parts, among them U28 74LS191, U29 74LS191, U38 74LS04, U41 74LS32, U48 74LS04, U6 74LS245, U77 74LS04

Commit message: Update
Parts:
- added C1 (x2), C6 (x2): 0.1uF, symbol Device:C
- added U26: 74LS04, symbol 74xx:74LS04
- added U53: 74LS32, symbol 74xx:74LS32
- renumbered U38 to U71, U48 to U71, U77 to U71, U41 to U72, U28 to U74, U29 to U75
Connections:
- net GND: now also C1.2, C1.2, C6.2, C6.2, U26.7 (GND), U53.7 (GND)
- net SB/S: now also U71.9; no longer U71.3
- net S/ADL: now also U71.1, U72.1; no longer U71.3, U72.2
- net S/SB: now also U71.5, U72.2; no longer U71.1, U72.1
- net VCC: now also U74.16 (VCC), U75.16 (VCC), C1.1, C1.1, C6.1, C6.1, U26.14 (VCC), U53.14 (VCC)
- net at U6.19 (CE): now also U71.6; no longer U71.4
- net at U74.11 (Pl), U75.11 (Pl): now also U71.8; no longer U71.4
- net at U74.13 (Rc): now also U75.14 (Cp)
- net at U72.3, U74.14 (Cp): no longer U75.14 (Cp)
- net S_DB_0 renamed S_ADL_0
- net S_DB_1 renamed S_ADL_1
- net S_DB_2 renamed S_ADL_2
- net S_DB_3 renamed S_ADL_3
- net S_DB_4 renamed S_ADL_4
- net S_DB_5 renamed S_ADL_5
- net S_DB_6 renamed S_ADL_6
- net S_DB_7 renamed S_ADL_7
Other:
- title: (none) -> Stack Pointer
- moved on the sheet: U71D
